File: RN2483.kicad_sch (KiCad schematic)
At the start: 3 parts

Commit message: Finishing schematic, first iteration of PCB
Parts:
- C10: renamed from C?; footprint (none) -> Capacitor_SMD:C_0805_2012Metric_Pad1.18x1.45mm_HandSolder
- J1: renamed from J?; footprint (none) -> Connector_Coaxial:SMA_Amphenol_132289_EdgeMount
- MODULE1: renamed from MODULE?; footprint MICROCHIP_RN2483-I/RM095 -> RN2483:RN2483A-I&slash_RM105
Changed lines of the file:
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@@
   (symbol (lib_id "power:GND") (at 172.72 130.81 0) (unit 1)
     (in_bom yes) (on_board yes) (fields_autoplaced)
-    (property "Reference" "#PWR?" (id 0) (at 172.72 137.16 0)
+    (property "Reference" "#PWR0128" (id 0) (at 172.72 137.16 0)
       (effects (font (size 1.27 1.27)) hide)
     )
@@
   (symbol (lib_id "AirQualitySensor1.2-rescue:RN2483-I_RM095-RN2483-I_RM095") (at 151.13 99.06 0) (unit 1)
     (in_bom yes) (on_board yes) (fields_autoplaced)
-    (property "Reference" "MODULE?" (id 0) (at 151.13 60.96 0))
+    (property "Reference" "MODULE1" (id 0) (at 151.13 60.96 0))
     (property "Value" "RN2483-I_RM095-RN2483-I_RM095" (id 1) (at 151.13 63.5 0))
-    (property "Footprint" "MICROCHIP_RN2483-I/RM095" (id 2) (at 151.13 99.06 0)
+    (property "Footprint" "RN2483:RN2483A-I&slash_RM105" (id 2) (at 151.13 99.06 0)
       (effects (font (size 1.27 1.27)) (justify left bottom) hide)
     )
@@
   (symbol (lib_id "Connector:Conn_Coaxial") (at 107.95 67.31 90) (unit 1)
     (in_bom yes) (on_board yes) (fields_autoplaced)
-    (property "Reference" "J?" (id 0) (at 108.2432 59.69 90))
+    (property "Reference" "J1" (id 0) (at 108.2432 59.69 90))
     (property "Value" "Conn_Coaxial" (id 1) (at 108.2432 62.23 90))
-    (property "Footprint" "" (id 2) (at 107.95 67.31 0)
+    (property "Footprint" "Connector_Coaxial:SMA_Amphenol_132289_EdgeMount" (id 2) (at 107.95 67.31 0)
       (effects (font (size 1.27 1.27)) hide)
     )
@@
   (symbol (lib_id "power:GND") (at 172.72 78.74 0) (unit 1)
     (in_bom yes) (on_board yes)
-    (property "Reference" "#PWR?" (id 0) (at 172.72 85.09 0)
+    (property "Reference" "#PWR0119" (id 0) (at 172.72 85.09 0)
       (effects (font (size 1.27 1.27)) hide)
     )
@@
   (symbol (lib_id "power:GND") (at 114.3 68.58 0) (unit 1)
     (in_bom yes) (on_board yes)
-    (property "Reference" "#PWR?" (id 0) (at 114.3 74.93 0)
+    (property "Reference" "#PWR0129" (id 0) (at 114.3 74.93 0)
       (effects (font (size 1.27 1.27)) hide)
     )
@@
   (symbol (lib_id "Device:C_Small") (at 172.72 74.93 0) (unit 1)
     (in_bom yes) (on_board yes) (fields_autoplaced)
-    (property "Reference" "C?" (id 0) (at 175.26 73.6662 0)
+    (property "Reference" "C10" (id 0) (at 175.26 73.6662 0)
       (effects (font (size 1.27 1.27)) (justify left))
     )
@@
       (effects (font (size 1.27 1.27)) (justify left))
     )
-    (property "Footprint" "" (id 2) (at 172.72 74.93 0)
+    (property "Footprint" "Capacitor_SMD:C_0805_2012Metric_Pad1.18x1.45mm_HandSolder" (id 2) (at 172.72 74.93 0)
       (effects (font (size 1.27 1.27)) hide)
     )
@@
   (symbol (lib_id "power:+3.3V") (at 172.72 67.31 0) (unit 1)
     (in_bom yes) (on_board yes) (fields_autoplaced)
-    (property "Reference" "#PWR?" (id 0) (at 172.72 71.12 0)
+    (property "Reference" "#PWR0126" (id 0) (at 172.72 71.12 0)
       (effects (font (size 1.27 1.27)) hide)
     )

Commit message: Small changes. Added BOM
Parts:
- MODULE1: footprint RN2483:RN2483A-I&slash_RM105 -> RF_Module:RN2483
Changed lines of the file:
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@@
     (property "Reference" "MODULE1" (id 0) (at 151.13 60.96 0))
     (property "Value" "RN2483-I_RM095-RN2483-I_RM095" (id 1) (at 151.13 63.5 0))
-    (property "Footprint" "RN2483:RN2483A-I&slash_RM105" (id 2) (at 151.13 99.06 0)
+    (property "Footprint" "RF_Module:RN2483" (id 2) (at 151.13 99.06 0)
       (effects (font (size 1.27 1.27)) (justify left bottom) hide)
     )

Commit message: Edited documentation
Other:
- title: (none) -> RN2483 LoRaWAN module
Changed lines of the file:
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@@
 (kicad_sch (version 20211123) (generator eeschema)
   (paper "A4")
+  (title_block
+    (title "RN2483 LoRaWAN module")
+    (date "2022-03-10")
+    (rev "1.0")
+  )
   (junction (at 172.72 71.12) (diameter 0) (color 0 0 0 0)
   )
