File: pwr.kicad_sch (KiCad schematic)
At the start: 6 parts

Commit message: Finishing schematic, first iteration of PCB
Parts:
- C11, C12, C13, C14: renamed from C?; footprint (none) -> Capacitor_SMD:C_0805_2012Metric_Pad1.18x1.45mm_HandSolder
- gave numbers to parts that had none: 2
Changed lines of the file:
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@@
   (symbol (lib_id "Device:C_Polarized_Small") (at 120.65 87.63 0) (unit 1)
     (in_bom yes) (on_board yes) (fields_autoplaced)
-    (property "Reference" "C?" (id 0) (at 123.19 85.8138 0)
+    (property "Reference" "C14" (id 0) (at 123.19 85.8138 0)
       (effects (font (size 1.27 1.27)) (justify left))
     )
@@
       (effects (font (size 1.27 1.27)) (justify left))
     )
-    (property "Footprint" "" (id 2) (at 120.65 87.63 0)
+    (property "Footprint" "Capacitor_SMD:C_0805_2012Metric_Pad1.18x1.45mm_HandSolder" (id 2) (at 120.65 87.63 0)
       (effects (font (size 1.27 1.27)) hide)
     )
@@
   (symbol (lib_id "LUYTSM:LD1117S33TR_SOT223") (at 107.95 34.29 0) (unit 1)
     (in_bom yes) (on_board yes) (fields_autoplaced)
-    (property "Reference" "U?" (id 0) (at 107.95 26.67 0))
+    (property "Reference" "U2" (id 0) (at 107.95 26.67 0))
     (property "Value" "LD1117S33TR_SOT223" (id 1) (at 107.95 29.21 0))
     (property "Footprint" "Package_TO_SOT_SMD:SOT-223-3_TabPin2" (id 2) (at 107.95 29.21 0)
@@
   (symbol (lib_id "Device:C_Polarized_Small") (at 120.65 39.37 0) (unit 1)
     (in_bom yes) (on_board yes) (fields_autoplaced)
-    (property "Reference" "C?" (id 0) (at 123.19 37.5538 0)
+    (property "Reference" "C13" (id 0) (at 123.19 37.5538 0)
       (effects (font (size 1.27 1.27)) (justify left))
     )
@@
       (effects (font (size 1.27 1.27)) (justify left))
     )
-    (property "Footprint" "" (id 2) (at 120.65 39.37 0)
+    (property "Footprint" "Capacitor_SMD:C_0805_2012Metric_Pad1.18x1.45mm_HandSolder" (id 2) (at 120.65 39.37 0)
       (effects (font (size 1.27 1.27)) hide)
     )
@@
   (symbol (lib_id "Device:C_Polarized_Small") (at 93.98 39.37 0) (unit 1)
     (in_bom yes) (on_board yes) (fields_autoplaced)
-    (property "Reference" "C?" (id 0) (at 96.52 37.5538 0)
+    (property "Reference" "C11" (id 0) (at 96.52 37.5538 0)
       (effects (font (size 1.27 1.27)) (justify left))
     )
@@
       (effects (font (size 1.27 1.27)) (justify left))
     )
-    (property "Footprint" "" (id 2) (at 93.98 39.37 0)
+    (property "Footprint" "Capacitor_SMD:C_0805_2012Metric_Pad1.18x1.45mm_HandSolder" (id 2) (at 93.98 39.37 0)
       (effects (font (size 1.27 1.27)) hide)
     )
@@
   (symbol (lib_id "Device:C_Polarized_Small") (at 93.98 87.63 0) (unit 1)
     (in_bom yes) (on_board yes) (fields_autoplaced)
-    (property "Reference" "C?" (id 0) (at 96.52 85.8138 0)
+    (property "Reference" "C12" (id 0) (at 96.52 85.8138 0)
       (effects (font (size 1.27 1.27)) (justify left))
     )
@@
       (effects (font (size 1.27 1.27)) (justify left))
     )
-    (property "Footprint" "" (id 2) (at 93.98 87.63 0)
+    (property "Footprint" "Capacitor_SMD:C_0805_2012Metric_Pad1.18x1.45mm_HandSolder" (id 2) (at 93.98 87.63 0)
       (effects (font (size 1.27 1.27)) hide)
     )
@@
   (symbol (lib_id "LUYTSM:LD1117S50TR_SOT223") (at 107.95 81.28 0) (unit 1)
     (in_bom yes) (on_board yes) (fields_autoplaced)
-    (property "Reference" "U?" (id 0) (at 107.95 73.66 0))
+    (property "Reference" "U3" (id 0) (at 107.95 73.66 0))
     (property "Value" "LD1117S50TR_SOT223" (id 1) (at 107.95 76.2 0))
     (property "Footprint" "Package_TO_SOT_SMD:SOT-223-3_TabPin2" (id 2) (at 107.95 76.2 0)
@@
   (symbol (lib_id "power:GND") (at 107.95 93.98 0) (unit 1)
     (in_bom yes) (on_board yes) (fields_autoplaced)
-    (property "Reference" "#PWR?" (id 0) (at 107.95 100.33 0)
+    (property "Reference" "#PWR0131" (id 0) (at 107.95 100.33 0)
       (effects (font (size 1.27 1.27)) hide)
     )
@@
   (symbol (lib_id "power:GND") (at 107.95 45.72 0) (unit 1)
     (in_bom yes) (on_board yes) (fields_autoplaced)
-    (property "Reference" "#PWR?" (id 0) (at 107.95 52.07 0)
+    (property "Reference" "#PWR0130" (id 0) (at 107.95 52.07 0)
       (effects (font (size 1.27 1.27)) hide)
     )

Commit message: Edited documentation
Other:
- title: (none) -> Power Regulators
Changed lines of the file:
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@@
 (kicad_sch (version 20211123) (generator eeschema)
   (paper "A5")
+  (title_block
+    (title "Power Regulators")
+    (date "2022-03-10")
+    (rev "1.0")
+  )
   (junction (at 93.98 44.45) (diameter 0) (color 0 0 0 0)
   )
